Commit message: New frame with slot for latch

File: urdf/door_fixed.urdf (robot description, URDF)
Before this commit: robot door_fixed, 5 links, 4 joints
Links:
- link frame: geometry collision mesh filename=package://door_fixed/meshes/frame(byKevin).stl; visual mesh filename=package://door_fixed/meshes/frame(byKevin).stl
